File: _autosave-pipsqueak_pcb.kicad_sch (KiCad schematic)
At the start: 118 parts, among them J1 Conn_01x02_Pin, J10 440054-2, J11 440054-2, J12 440054-2, J13 Conn_01x04_Pin, J14 440054-2, J15 440054-2, J16 Conn_01x04_Pin, J18 Conn_01x04_Pin, J19 10118192-0002LF, J2 Conn_01x02_Pin, J20 Conn_01x04_Pin, J21 3PinHeader, J22 3PinHeader, J3 Conn_01x01_Pin, J4 Conn_01x08_Pin, J5 Conn_01x04_Pin, J6 Conn_01x04_Pin, J7 Conn_01x02_Pin, J8 Conn_01x02_Pin, J9 440054-2, Q1 CSD18535KCS, Q2 MMBT3904, Q3 MMBT3904, U1 SUP90P06-09L-E3 or MCP80P06Y-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, U10 FT231XS-R, U2 MCP1402T-E_OT, U3 MP1584EN, U4 TMC2209_SILENTSTEPSTICK, U5 ESP32-WROOM-32E-N8, U6 TMC2209_SILENTSTEPSTICK, U7 TMC2209_SILENTSTEPSTICK, U8 TMC2209_SILENTSTEPSTICK

Commit message: schematic finished
Parts:
- removed J3: Conn_01x01_Pin, Connector_PinHeader_2.54mm:PinHeader_1x01_P2.54mm_Vertical, symbol Connector:Conn_01x01_Pin
- added C? (x2): 0.1uF, Capacitor_SMD:C_0603_1608Metric, symbol Device:C
- added C?: 0.1uF, Capacitor_SMD:C_1206_3216Metric, symbol Device:C
- added C?: 220uF, Capacitor_SMD:C_Elec_6.3x7.7, symbol Device:C_Polarized
- added J? (x2): Conn_01x04_Pin, Connector_JST:JST_XH_B4B-XH-A_1x04_P2.50mm_Vertical, symbol Connector:Conn_01x04_Pin
- added J? (x2): Conn_01x04_Pin, Connector_PinHeader_2.54mm:PinHeader_1x04_P2.54mm_Vertical, symbol Connector:Conn_01x04_Pin
- added J?: Conn_01x02_Pin, Connector_PinHeader_2.54mm:PinHeader_1x02_P2.54mm_Vertical, symbol Connector:Conn_01x02_Pin
- added R? (x2): 100, Resistor_SMD:R_0805_2012Metric, symbol Device:R
- added R? (x2): 0, Resistor_SMD:R_1210_3225Metric_Pad1.30x2.65mm_HandSolder, symbol Device:R
- added R?: 1k, Resistor_SMD:R_0603_1608Metric, symbol Device:R
- added R?: 20k, Resistor_SMD:R_0603_1608Metric, symbol Device:R
- added R?: 10k, Resistor_SMD:R_0603_1608Metric, symbol Device:R
Connections:
- net +3V3: now also C?.1, J?.4 (Pin_4)
- net +5V: now also C?.1, C?.2, C?.2, J?.1 (Pin_1)
- net ESP32RXD: now also J?.2 (Pin_2), J?.2 (Pin_2), J?.4 (Pin_4), J?.4 (Pin_4), R?.2
- net ESP32TXD: now also J?.1 (Pin_1), J?.3 (Pin_3), J?.3 (Pin_3), R?.2
- net GND: now also C?.1, C?.1, C?.2, C?.2, J?.1 (Pin_1), J?.4 (Pin_4), R?.2
- net IO17: now also R?.2
- net IO18: now also R?.2
- net IO19: now also J?.1 (Pin_1)
- net IO21: now also J?.2 (Pin_2)
- net IO22: no longer R?.2, U5.36 (IO22), U?.27 (SDA)
- net at J21.3: now also U?.22 (LED15)
- net at J?.3: now also U?.18 (LED11)
- net at J22.3: now also U?.20 (LED13)
- net at J?.3: now also U?.16 (LED9)
- net at U?.13 (LED7): now also J?.3
- net IO23 renamed SCL
- new net: J?.2 (Pin_2), R?.1 (x2)
- new net: R?.1, R?.1, R?.2
- new net: J?.3 (Pin_3), R?.1 (x2)
- new net: R?.1, R?.2
- new net SDA: R?.2, U5.36 (IO22), U?.27 (SDA)
Other:
- note added: "NX4827P043-011C Touchscreen"
- moved on the sheet: C1, C10, C11, C12, C18, C19, C6, C7, C8, C9, C?, J10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
