File: _autosave-pipsqueak_pcb.kicad_pcb (KiCad board)
At the start: 2 copper layers, 175 x 91 mm, 135 parts, among them J1 Conn_01x02_Pin, J10 Conn_01x02_Pin, J11 440054-2, J12 440054-2, J13 440054-2, J14 Conn_01x04_Pin, J15 440054-2, J16 440054-2, J17 440054-2, J18 Conn_01x04_Pin, J19 3PinHeader, J2 Conn_01x02_Pin, J20 3PinHeader, J21 3PinHeader, J22 Conn_01x04_Pin, J24 3PinHeader, J25 10118192-0002LF, J26 Conn_01x04_Pin, J27 3PinHeader, J28 Conn_01x04_Pin, J29 Conn_01x04_Pin, J3 Conn_01x02_Pin, J4 Conn_01x04_Pin, J5 Conn_01x08_Pin, J6 Conn_01x04_Pin, J7 Conn_01x04_Pin, J8 Conn_01x04_Pin, J9 Conn_01x02_Pin, Q1 CSD18535KCS, Q2 MMBT3904, Q3 MMBT3904, U1 SUP90P06-09L-E3 or MCP80P06Y-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, U10 FT231XS-R, U2 MCP1402T-E_OT, U3 MP1584EN, U4 TMC2209_SILENTSTEPSTICK, U5 ESP32-WROOM-32E-N8, U6 TMC2209_SILENTSTEPSTICK, U7 TMC2209_SILENTSTEPSTICK, U8 PCA9685PW, U9 TMC2209_SILENTSTEPSTICK

Commit message: finished
Other:
- board text added: "Nostopharma X Blu Cru 6417"
Changed lines of the file:
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@@
 		)
 	)
-	(gr_text "Blu Cru 6417"
-		(at 95 51.5 0)
+	(gr_text "Nostopharma X Blu Cru 6417"
+		(at 95 48 0)
 		(layer "B.SilkS")
 		(effects
@@
 	)
 	(gr_text "Cooper Li 5/13/26"
-		(at 95 47.5 0)
+		(at 95 52 0)
 		(layer "B.SilkS")
 		(effects
