File: pipsqueak_pcb.kicad_sch (KiCad schematic)
At the start: 118 parts, among them J1 Conn_01x02_Pin, J10 440054-2, J11 440054-2, J12 440054-2, J13 Conn_01x04_Pin, J14 440054-2, J15 440054-2, J16 Conn_01x04_Pin, J18 Conn_01x04_Pin, J19 10118192-0002LF, J2 Conn_01x02_Pin, J20 Conn_01x04_Pin, J21 3PinHeader, J22 3PinHeader, J3 Conn_01x01_Pin, J4 Conn_01x08_Pin, J5 Conn_01x04_Pin, J6 Conn_01x04_Pin, J7 Conn_01x02_Pin, J8 Conn_01x02_Pin, J9 440054-2, Q1 CSD18535KCS, Q2 MMBT3904, Q3 MMBT3904, U1 SUP90P06-09L-E3 or MCP80P06Y-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, U10 FT231XS-R, U2 MCP1402T-E_OT, U3 MP1584EN, U4 TMC2209_SILENTSTEPSTICK, U5 ESP32-WROOM-32E-N8, U6 TMC2209_SILENTSTEPSTICK, U7 TMC2209_SILENTSTEPSTICK, U8 TMC2209_SILENTSTEPSTICK

Commit message: pca fix
Parts:
- removed J3: Conn_01x01_Pin, Connector_PinHeader_2.54mm:PinHeader_1x01_P2.54mm_Vertical, symbol Connector:Conn_01x01_Pin
- added C? (x2): 0.1uF, Capacitor_SMD:C_0603_1608Metric, symbol Device:C
- added C?: 10uF, Capacitor_SMD:C_1206_3216Metric, symbol Device:C
- added C?: 220uF, Capacitor_SMD:C_Elec_6.3x7.7, symbol Device:C_Polarized
- added J? (x2): Conn_01x04_Pin, Connector_JST:JST_XH_B4B-XH-A_1x04_P2.50mm_Vertical, symbol Connector:Conn_01x04_Pin
- added J? (x2): Conn_01x04_Pin, Connector_PinHeader_2.54mm:PinHeader_1x04_P2.54mm_Vertical, symbol Connector:Conn_01x04_Pin
- added J?: Conn_01x02_Pin, Connector_PinHeader_2.54mm:PinHeader_1x02_P2.54mm_Vertical, symbol Connector:Conn_01x02_Pin
- added R? (x2): 100, Resistor_SMD:R_0805_2012Metric, symbol Device:R
- added R? (x2): 0, Resistor_SMD:R_1210_3225Metric_Pad1.30x2.65mm_HandSolder, symbol Device:R
- added R?: 1k, Resistor_SMD:R_0603_1608Metric, symbol Device:R
- added R?: 20k, Resistor_SMD:R_0603_1608Metric, symbol Device:R
- added R?: 10k, Resistor_SMD:R_0603_1608Metric, symbol Device:R
Connections:
- net +3V3: now also C?.1, J?.4 (Pin_4)
- net +5V: now also C?.1, C?.2, C?.2, J?.1 (Pin_1)
- net ESP32RXD: now also J?.2 (Pin_2), J?.4 (Pin_4), R?.2
- net ESP32TXD: now also J?.1 (Pin_1), J?.3 (Pin_3), R?.2
- net GND: now also U?.1 (A0), U?.2 (A1), U?.23 (~{OE}), U?.24 (A5), U?.3 (A2), U?.4 (A3), U?.5 (A4), C?.1, C?.1, C?.2, C?.2, J?.1 (Pin_1), J?.4 (Pin_4), R?.2
- net IO17: now also R?.2
- net IO18: now also R?.2
- net IO19: now also J?.1 (Pin_1)
- net IO21: now also J?.2 (Pin_2)
- net at J21.3: now also U?.22 (LED15)
- net at J?.3: now also U?.18 (LED11)
- net at J22.3: now also U?.20 (LED13)
- net at J?.3: now also U?.16 (LED9)
- net at U?.13 (LED7): now also J?.3
- net IO22 renamed SDA
- net SDA: now also J?.1 (Pin_1), J?.3 (Pin_3)
- net IO23 renamed SCL
- net SCL: now also J?.2 (Pin_2), J?.4 (Pin_4)
- new net: J?.2 (Pin_2), R?.1 (x2)
- new net: R?.1, R?.1, R?.2
- new net: J?.3 (Pin_3), R?.1 (x2)
- new net: R?.1, R?.2
Other:
- note added: "NX4827P043-011C Touchscreen"
- note removed: "TODO: UART+I2C breakouts"
- moved on the sheet: C1, C10, C11, C12, C18, C19, C6, C7, C8, C9, C?, J10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

Commit message: finished
Parts:
- added C1: 1uF, Capacitor_SMD:C_0805_2012Metric, symbol Device:C
- added C47: 0.1uF, Capacitor_SMD:C_0603_1608Metric, symbol Device:C
- C6: renamed from C4; value 220uF -> 1000uF; footprint Capacitor_SMD:C_Elec_6.3x7.7 -> Capacitor_SMD:C_Elec_10x10.2
- J1, J2: footprint Connector_AMASS:AMASS_XT30U-F_1x02_P5.0mm_Vertical -> Connector_AMASS:AMASS_XT30UPB-M_1x02_P5.0mm_Vertical
- R18: renamed from R12; footprint Resistor_SMD:R_0603_1608Metric -> Resistor_SMD:R_1206_3216Metric
- R23, R26: renamed from R?; footprint Resistor_SMD:R_0805_2012Metric -> Resistor_SMD:R_0603_1608Metric
- gave numbers to parts that had none: 31
- renumbered C10 to C12, C7 to C13, C9 to C14, C11 to C15, C12 to C16, C18 to C17, C19 to C18, C13 to C19, C1 to C2, C14 to C20, C15 to C21, C34 to C22, C35 to C23, C16 to C25, C36 to C26, C37 to C27, C17 to C29, C2 to C3, C20 to C30, C24 to C33, C25 to C34, C26 to C35, C27 to C36, C21 to C37, C22 to C39, C3 to C4, C28 to C40, C23 to C41, C29 to C44, C30 to C45, C31 to C48, C32 to C49, C6 to C5, C33 to C51, C38 to C52, C8 to C7, C5 to C8, J8 to J10, J9 to J11, J10 to J12, J11 to J13, J12 to J15, J14 to J16, J15 to J17, J13 to J18, J21 to J19, J22 to J20, J16 to J22, J17 to J23, J19 to J25, J18 to J26, J20 to J28, J4 to J5, J5 to J6, J6 to J7, J7 to J9, R9 to R10, R7 to R11, R10 to R15, R13 to R16, R11 to R17, R14 to R19, R18 to R24, R19 to R25, R20 to R27, R16 to R30, R17 to R31, R8 to R9, U8 to U9
Connections:
- net +24V: now also C21.2
- net +3V3: now also U4.15 (MS1), U6.15 (MS1), U7.15 (MS1), U9.15 (MS1)
- net +5V: now also C1.1
- net GND: now also C1.2, C47.1; no longer U4.15 (MS1), U6.15 (MS1), U7.15 (MS1), U9.15 (MS1)
- net IO34: now also C7.1, J13.2, R15.1; no longer C5.1, J12.2, R10.1
- net IO35: now also C12.1, J15.2, R16.1; no longer C4.1, J11.2, R9.1
- net IO36: now also C4.1, J11.2, R9.1; no longer C7.1, J13.2, R15.1
- net IO39: now also C5.1, J12.2, R10.1; no longer C12.1, J15.2, R16.1
- net SCL: now also U5.36 (IO22); no longer U5.37 (IO23)
- net SDA: now also U5.37 (IO23); no longer U5.36 (IO22)
- net at C44.1, R27.2, U10.13 (3V3OUT): now also C47.2
- net M1B: now reaches U4.3 (M1B)
- net M1B: now also J18.4 (Pin_4); no longer J18.2 (Pin_2)
- net M1A: now reaches U4.4 (M1A)
- net M1A: now also J18.3 (Pin_3); no longer J18.4 (Pin_4)
- net M2A: now reaches U4.5 (M2A)
- net M2A: now also J18.2 (Pin_2); no longer J18.3 (Pin_3)
- net M2B: now reaches J18.1 (Pin_1), U4.6 (M2B)
- net at J22.2 (Pin_2): now also U6.5 (M2A); no longer U6.3 (M1B)
- net at J22.3 (Pin_3): now also U6.4 (M1A); no longer U6.5 (M2A)
- net at J22.4 (Pin_4): now also U6.3 (M1B); no longer U6.4 (M1A)
- net at J26.2 (Pin_2): now also U7.5 (M2A); no longer U7.3 (M1B)
- net at J26.3 (Pin_3): now also U7.4 (M1A); no longer U7.5 (M2A)
- net at J26.4 (Pin_4): now also U7.3 (M1B); no longer U7.4 (M1A)
- net at J28.2 (Pin_2): now also U9.5 (M2A); no longer U9.3 (M1B)
- net at J28.3 (Pin_3): now also U9.4 (M1A); no longer U9.5 (M2A)
- net at J28.4 (Pin_4): now also U9.3 (M1B); no longer U9.4 (M1A)
Other:
- note added: "Default Connect"
- note added: "Default NC"
- moved on the sheet: C2, J18, J22, J26, J28, R27, U2
